File: Experiments/SAMD11 Feather 24QFN.sch (EAGLE design)
At the start: 34 parts, among them IC1 ATSAMD11D14A-MUT, J1 10118193-0001LF, Q1 DMG341, SW1 SPST_TACT-KMR2, U1 AP2112-3.3, U2 MCP73831T-2ACI/OT, X1 JSTPH, X2 2x5 0.05" SWD

Commit message: fix swdio/swclk mixup
Connections:
- net SWCLK: now also IC1.PA30; no longer IC1.PA31
- net SWDIO: now also IC1.PA31; no longer IC1.PA30
Changed lines of the file:
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@@
 <part name="SW1" library="adafruit" deviceset="SPST_TACT" device="-KMR2" value="SPST_TACT-KMR2"/>
 <part name="SWCLK" library="testpad" library_urn="urn:adsk.eagle:library:385" deviceset="TPSQ" device="TP20R" package3d_urn="urn:adsk.eagle:package:27973/1"/>
-<part name="SWDIO" library="testpad" library_urn="urn:adsk.eagle:library:385" deviceset="TPSQ" device="TP20R" package3d_urn="urn:adsk.eagle:package:27973/1"/>
 <part name="FRAME1" library="My Stuff" deviceset="A4L-LOC" device=""/>
 <part name="GND22" library="supply1" library_urn="urn:adsk.eagle:library:371" deviceset="GND" device=""/>
@@
 <part name="FID3" library="microbuilder" deviceset="FIDUCIAL" device="_1MM"/>
 <part name="FID4" library="microbuilder" deviceset="FIDUCIAL" device="_1MM"/>
+<part name="SWDIO" library="testpad" library_urn="urn:adsk.eagle:library:385" deviceset="TPSQ" device="TP20R" package3d_urn="urn:adsk.eagle:package:27973/1"/>
 </parts>
 <sheets>
@@
 <attribute name="VALUE" x="125.73" y="156.845" size="1.778" layer="96" rot="R270"/>
 </instance>
-<instance part="SWCLK" gate="G$1" x="86.36" y="71.12" smashed="yes" rot="R90">
-<attribute name="TP_SIGNAL_NAME" x="87.63" y="73.66" size="1.778" layer="97" rot="R90"/>
-</instance>
-<instance part="SWDIO" gate="G$1" x="86.36" y="73.66" smashed="yes" rot="R90">
+<instance part="SWCLK" gate="G$1" x="86.36" y="73.66" smashed="yes" rot="R90">
 <attribute name="TP_SIGNAL_NAME" x="87.63" y="76.2" size="1.778" layer="97" rot="R90"/>
 </instance>
@@
 <instance part="FID3" gate="G$1" x="302.26" y="58.42" smashed="yes"/>
 <instance part="FID4" gate="G$1" x="297.18" y="58.42" smashed="yes"/>
+<instance part="SWDIO" gate="G$1" x="86.36" y="71.12" smashed="yes" rot="R90">
+<attribute name="TP_SIGNAL_NAME" x="87.63" y="73.66" size="1.778" layer="97" rot="R90"/>
+</instance>
 </instances>
 <busses>
@@
 </segment>
 <segment>
-<wire x1="71.12" y1="73.66" x2="83.82" y2="73.66" width="0.1524" layer="91"/>
-<label x="73.66" y="73.66" size="1.778" layer="95"/>
-<pinref part="IC1" gate="G$1" pin="PA30"/>
+<wire x1="71.12" y1="71.12" x2="83.82" y2="71.12" width="0.1524" layer="91"/>
 <pinref part="SWDIO" gate="G$1" pin="TP"/>
+<pinref part="IC1" gate="G$1" pin="PA31"/>
+<label x="73.66" y="71.12" size="1.778" layer="95"/>
 </segment>
 </net>
@@
 </segment>
 <segment>
-<wire x1="71.12" y1="71.12" x2="83.82" y2="71.12" width="0.1524" layer="91"/>
-<label x="73.66" y="71.12" size="1.778" layer="95"/>
-<pinref part="IC1" gate="G$1" pin="PA31"/>
+<label x="73.66" y="73.66" size="1.778" layer="95"/>
 <pinref part="SWCLK" gate="G$1" pin="TP"/>
-</segment>
-</net>
+<pinref part="IC1" gate="G$1" pin="PA30"/>
+<wire x1="71.12" y1="73.66" x2="83.82" y2="73.66" width="0.1524" layer="91"/>
+</segment>
+</net>
