File: OSO Curriculum/OSO-SAFE-C1-02.brd (EAGLE design)
At the start: 50.8 x 22.9 mm, 19 parts, among them U1 LM1117T-3.3, U2 ATSAMD11D14A-SSNT

Commit message: scoot usb breakout up a bit
Parts:
- moved USB 1.30 mm to (8.38, 12.7)
Routing:
- net VBUS: track 31.4 -> 32.2 mm
Other:
- board text added: "OSO-SAFE-C1-02"
- board text removed: "OSO-SAFE-C1-01"
Changed lines of the file:
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@@
 <layer number="14" name="Route14" color="1" fill="6" visible="no" active="no"/>
 <layer number="15" name="Route15" color="4" fill="6" visible="no" active="no"/>
-<layer number="16" name="Bottom" color="1" fill="1" visible="no" active="yes"/>
+<layer number="16" name="Bottom" color="1" fill="1" visible="yes" active="yes"/>
 <layer number="17" name="Pads" color="2" fill="1" visible="yes" active="yes"/>
 <layer number="18" name="Vias" color="2" fill="1" visible="yes" active="yes"/>
@@
 <layer number="20" name="Dimension" color="15" fill="1" visible="yes" active="yes"/>
 <layer number="21" name="tPlace" color="14" fill="1" visible="yes" active="yes"/>
-<layer number="22" name="bPlace" color="13" fill="1" visible="no" active="yes"/>
+<layer number="22" name="bPlace" color="13" fill="1" visible="yes" active="yes"/>
 <layer number="23" name="tOrigins" color="14" fill="1" visible="yes" active="yes"/>
-<layer number="24" name="bOrigins" color="13" fill="1" visible="no" active="yes"/>
+<layer number="24" name="bOrigins" color="13" fill="1" visible="yes" active="yes"/>
 <layer number="25" name="tNames" color="7" fill="1" visible="yes" active="yes"/>
-<layer number="26" name="bNames" color="7" fill="1" visible="no" active="yes"/>
+<layer number="26" name="bNames" color="7" fill="1" visible="yes" active="yes"/>
 <layer number="27" name="tValues" color="11" fill="1" visible="no" active="yes"/>
 <layer number="28" name="bValues" color="7" fill="1" visible="no" active="yes"/>
@@
 <layer number="38" name="bTest" color="7" fill="1" visible="no" active="yes"/>
 <layer number="39" name="tKeepout" color="4" fill="11" visible="yes" active="yes"/>
-<layer number="40" name="bKeepout" color="1" fill="11" visible="no" active="yes"/>
+<layer number="40" name="bKeepout" color="1" fill="11" visible="yes" active="yes"/>
 <layer number="41" name="tRestrict" color="4" fill="10" visible="yes" active="yes"/>
-<layer number="42" name="bRestrict" color="1" fill="10" visible="no" active="yes"/>
-<layer number="43" name="vRestrict" color="2" fill="10" visible="no" active="yes"/>
+<layer number="42" name="bRestrict" color="1" fill="10" visible="yes" active="yes"/>
+<layer number="43" name="vRestrict" color="2" fill="10" visible="yes" active="yes"/>
 <layer number="44" name="Drills" color="7" fill="1" visible="no" active="yes"/>
 <layer number="45" name="Holes" color="7" fill="1" visible="no" active="yes"/>
@@
 <layer number="50" name="dxf" color="7" fill="1" visible="no" active="no"/>
 <layer number="51" name="tDocu" color="7" fill="1" visible="yes" active="yes"/>
-<layer number="52" name="bDocu" color="7" fill="1" visible="no" active="yes"/>
+<layer number="52" name="bDocu" color="7" fill="1" visible="yes" active="yes"/>
 <layer number="53" name="tGND_GNDA" color="7" fill="9" visible="no" active="no"/>
 <layer number="54" name="bGND_GNDA" color="1" fill="9" visible="no" active="no"/>
@@
 the Book
 #4</text>
-<text x="9.906" y="21.59" size="0.8128" layer="22" font="vector" ratio="18" rot="MR180" align="center">OSO-SAFE-C1-01</text>
-<rectangle x1="0.254" y1="1.27" x2="10.414" y2="21.59" layer="43"/>
+<text x="9.906" y="21.59" size="0.8128" layer="22" font="vector" ratio="18" rot="MR180" align="center">OSO-SAFE-C1-02</text>
+<rectangle x1="0" y1="2.54" x2="10.16" y2="22.86" layer="43"/>
 <text x="25.527" y="21.59" size="0.635" layer="21" font="vector" ratio="12" rot="R90" align="center">SWCL</text>
 <text x="25.527" y="1.27" size="0.635" layer="21" font="vector" ratio="12" rot="R90" align="center">PA07</text>
-<text x="6.477" y="16.51" size="0.635" layer="21" font="vector" ratio="18" rot="R270" align="center">VBUS</text>
-<text x="6.477" y="13.97" size="0.635" layer="21" font="vector" ratio="18" rot="R270" align="center">D-</text>
-<text x="6.477" y="11.43" size="0.635" layer="21" font="vector" ratio="18" rot="R270" align="center">D+</text>
-<text x="6.477" y="6.35" size="0.635" layer="21" font="vector" ratio="18" rot="R270" align="center">GND</text>
-<text x="10.795" y="16.51" size="0.635" layer="22" font="vector" ratio="18" rot="SMR270" align="center">VBUS</text>
-<text x="10.795" y="13.97" size="0.635" layer="22" font="vector" ratio="18" rot="SMR270" align="center">D-</text>
-<text x="10.795" y="11.43" size="0.635" layer="22" font="vector" ratio="18" rot="SMR270" align="center">D+</text>
-<text x="10.795" y="6.35" size="0.635" layer="22" font="vector" ratio="18" rot="SMR270" align="center">GND</text>
+<text x="6.223" y="17.78" size="0.635" layer="21" font="vector" ratio="18" rot="R270" align="center">VBUS</text>
+<text x="6.223" y="15.24" size="0.635" layer="21" font="vector" ratio="18" rot="R270" align="center">D-</text>
+<text x="6.223" y="12.7" size="0.635" layer="21" font="vector" ratio="18" rot="R270" align="center">D+</text>
+<text x="6.223" y="7.62" size="0.635" layer="21" font="vector" ratio="18" rot="R270" align="center">GND</text>
+<text x="10.541" y="17.78" size="0.635" layer="22" font="vector" ratio="18" rot="SMR270" align="center">VBUS</text>
+<text x="10.541" y="15.24" size="0.635" layer="22" font="vector" ratio="18" rot="SMR270" align="center">D-</text>
+<text x="10.541" y="12.7" size="0.635" layer="22" font="vector" ratio="18" rot="SMR270" align="center">D+</text>
+<text x="10.541" y="7.62" size="0.635" layer="22" font="vector" ratio="18" rot="SMR270" align="center">GND</text>
 <text x="26.416" y="20.574" size="0.6096" layer="22" font="vector" ratio="12" rot="SMR270" align="center-left">PA30/SWCLK</text>
 <text x="29.21" y="20.574" size="0.6096" layer="22" font="vector" ratio="12" rot="SMR270" align="center-left">PA08</text>
@@
 <attribute name="VENDOR" value="Texas Instruments" x="12.446" y="11.43" size="1.778" layer="27" rot="R90" display="off"/>
 </element>
-<element name="USB" library="pinhead" library_urn="urn:adsk.eagle:library:325" package="1X05" package3d_urn="urn:adsk.eagle:package:22469/2" value="" x="8.636" y="11.43" smashed="yes" rot="R270">
-<attribute name="VALUE" x="5.461" y="17.78" size="1.27" layer="27" rot="R270"/>
+<element name="USB" library="pinhead" library_urn="urn:adsk.eagle:library:325" package="1X05" package3d_urn="urn:adsk.eagle:package:22469/2" value="" x="8.382" y="12.7" smashed="yes" rot="R270">
+<attribute name="VALUE" x="5.207" y="19.05" size="1.27" layer="27" rot="R270"/>
 </element>
 <element name="R2" library="adafruit" package="0207/9" value="1K" x="24.892" y="14.732" smashed="yes" rot="R270">
@@
 <contactref element="R1" pad="2"/>
 <wire x1="13.462" y1="11.43" x2="17.018" y2="14.986" width="0.3048" layer="16"/>
-<wire x1="11.938" y1="14.986" x2="10.414" y2="16.51" width="0.3048" layer="1"/>
-<wire x1="10.414" y1="16.51" x2="8.636" y2="16.51" width="0.3048" layer="1"/>
+<wire x1="11.938" y1="14.986" x2="9.144" y2="17.78" width="0.3048" layer="1"/>
+<wire x1="9.144" y1="17.78" x2="8.382" y2="17.78" width="0.3048" layer="1"/>
 <wire x1="11.938" y1="14.986" x2="17.018" y2="14.986" width="0.3048" layer="1"/>
 <wire x1="21.59" y1="21.59" x2="21.59" y2="19.558" width="0.3048" layer="1"/>
@@
 <signal name="USB_P">
 <contactref element="U2" pad="15"/>
-<wire x1="35.4584" y1="12.827" x2="23.2664" y2="12.827" width="0.254" layer="1"/>
-<wire x1="23.2664" y1="12.827" x2="22.7748375" y2="13.3185625" width="0.254" layer="1"/>
-<wire x1="10.414" y1="11.43" x2="12.3025625" y2="13.3185625" width="0.254" layer="1"/>
-<wire x1="12.3025625" y1="13.3185625" x2="22.7748375" y2="13.3185625" width="0.254" layer="1"/>
+<wire x1="35.4584" y1="12.827" x2="34.4424" y2="12.827" width="0.254" layer="1"/>
+<wire x1="34.4424" y1="12.827" x2="33.9508375" y2="13.3185625" width="0.254" layer="1"/>
+<wire x1="10.16" y1="12.7" x2="10.7785625" y2="13.3185625" width="0.254" layer="1"/>
+<wire x1="10.7785625" y1="13.3185625" x2="33.9508375" y2="13.3185625" width="0.254" layer="1"/>
 <contactref element="USB" pad="3"/>
-<wire x1="8.636" y1="11.43" x2="10.414" y2="11.43" width="0.254" layer="1"/>
+<wire x1="8.382" y1="12.7" x2="10.16" y2="12.7" width="0.254" layer="1"/>
 </signal>
 <signal name="USB_N">
 <contactref element="U2" pad="14"/>
-<wire x1="28.8544" y1="14.097" x2="35.4584" y2="14.097" width="0.254" layer="1"/>
-<wire x1="27.7114" y1="15.24" x2="28.8544" y2="14.097" width="0.254" layer="1"/>
-<wire x1="23.955384375" y1="15.24" x2="27.7114" y2="15.24" width="0.254" layer="1"/>
-<wire x1="22.685384375" y1="13.97" x2="23.955384375" y2="15.24" width="0.254" layer="1"/>
 <contactref element="USB" pad="2"/>
-<wire x1="8.636" y1="13.97" x2="22.685384375" y2="13.97" width="0.254" layer="1"/>
+<wire x1="11.049" y1="14.097" x2="9.906" y2="15.24" width="0.254" layer="1"/>
+<wire x1="8.382" y1="15.24" x2="9.906" y2="15.24" width="0.254" layer="1"/>
+<wire x1="35.4584" y1="14.097" x2="11.049" y2="14.097" width="0.254" layer="1"/>
 </signal>
 <signal name="PA05">
