File: OSO Curriculum/OSO-SAFE-C1-02.brd (EAGLE design)
At the start: 50.8 x 22.9 mm, 19 parts, among them U1 LM1117T-3.3, U2 ATSAMD11D14A-SSNT

Commit message: update SAMD11 feathers
Parts:
- removed U1: LM1117T-3.3, My Stuff:T03B
- added U3: MCP1700-3302E/TO, MCP1700-3302E_TO:TO127P254X495-3
- moved U$9 0.25 mm to (3.56, 11.2)
Connections:
- net +3V3: now also U3.3; no longer U1.2
- net GND: now also U3.1; no longer U1.1
- net VBUS: now also U3.2; no longer U1.3
Routing:
- net VBUS: track 32.2 -> 31.4 mm
Changed lines of the file:
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@@
 <layer number="27" name="tValues" color="11" fill="1" visible="no" active="yes"/>
 <layer number="28" name="bValues" color="7" fill="1" visible="no" active="yes"/>
-<layer number="29" name="tStop" color="7" fill="3" visible="no" active="yes"/>
+<layer number="29" name="tStop" color="7" fill="3" visible="yes" active="yes"/>
 <layer number="30" name="bStop" color="7" fill="6" visible="no" active="yes"/>
 <layer number="31" name="tCream" color="7" fill="4" visible="no" active="yes"/>
@@
 <attribute name="VALUE" x="43.0784" y="17.9578" size="0.508" layer="27" font="vector" ratio="18" rot="SR180" align="center"/>
 </element>
-<element name="U1" library="My Stuff" package="T03B" value="LM1117T-3.3" x="12.446" y="11.43" smashed="yes" rot="R90">
-<attribute name="BUILT_BY" value="EMA_UL_Team" x="12.446" y="11.43" size="1.778" layer="27" rot="R90" display="off"/>
-<attribute name="MANUFACTURER_PART_NUMBER" value="LM1117T-3.3/NOPB" x="12.446" y="11.43" size="1.778" layer="27" rot="R90" display="off"/>
-<attribute name="NAME" x="14.2494" y="3.81" size="0.508" layer="51" font="vector" ratio="18" rot="SR0"/>
-<attribute name="VENDOR" value="Texas Instruments" x="12.446" y="11.43" size="1.778" layer="27" rot="R90" display="off"/>
-</element>
 <element name="USB" library="pinhead" library_urn="urn:adsk.eagle:library:325" package="1X05" package3d_urn="urn:adsk.eagle:package:22469/2" value="" x="8.382" y="12.7" smashed="yes" rot="R270">
 <attribute name="VALUE" x="5.207" y="19.05" size="1.27" layer="27" rot="R270"/>
@@
 </element>
 <element name="U$8" library="My Stuff" package="OSO_WORDMARK_ONELINE_725MIL_1000DPI" value="" x="46.99" y="20.574" smashed="yes" rot="MR270"/>
-<element name="U$9" library="My Stuff" package="OSO_BEAR_250X360MIL_1000DPI" value="" x="3.81" y="11.176" smashed="yes" rot="MR0"/>
+<element name="U$9" library="My Stuff" package="OSO_BEAR_250X360MIL_1000DPI" value="" x="3.556" y="11.176" smashed="yes" rot="MR0"/>
 <element name="U$10" library="microbuilder" package="MOUNTINGHOLE_2.5_PLATED" value="MOUNTINGHOLE2.5" x="2.54" y="20.32" smashed="yes">
 <attribute name="BOM" value="EXCLUDE" x="2.54" y="20.32" size="0.508" layer="27" font="vector" ratio="18" display="off"/>
+</element>
+<element name="U3" library="MCP1700-3302E_TO" package="TO127P254X495-3" value="MCP1700-3302E/TO" x="14.478" y="9.398" smashed="yes" rot="R270">
+<attribute name="DESCRIPTION" value=" Linear Voltage Regulator IC 1 Output 250mA TO-92-3 " x="14.478" y="9.398" size="1.778" layer="27" rot="R270" display="off"/>
+<attribute name="DIGI-KEY_PART_NUMBER" value="MCP1700-3302E/TO-ND" x="14.478" y="9.398" size="1.778" layer="27" rot="R270" display="off"/>
+<attribute name="DIGI-KEY_PURCHASE_URL" value="https://www.digikey.com/product-detail/en/microchip-technology/MCP1700-3302E-TO/MCP1700-3302E-TO-ND/652680?utm_source=snapeda&amp;utm_medium=aggregator&amp;utm_campaign=symbol" x="14.478" y="9.398" size="1.778" layer="27" rot="R270" display="off"/>
+<attribute name="MF" value="Microchip" x="14.478" y="9.398" size="1.778" layer="27" rot="R270" display="off"/>
+<attribute name="MP" value="MCP1700-3302E/TO" x="14.478" y="9.398" size="1.778" layer="27" rot="R270" display="off"/>
+<attribute name="NAME" x="13.208" y="7.62" size="0.508" layer="25" font="vector" ratio="18" rot="SR0" align="center"/>
+<attribute name="PACKAGE" value="TO-92 Microchip" x="14.478" y="9.398" size="1.778" layer="27" rot="R270" display="off"/>
+<attribute name="VALUE" x="8.77423125" y="16.171240625" size="2.087990625" layer="27" ratio="10" rot="SR270"/>
 </element>
 </elements>
@@
 <contactref element="JP1" pad="13"/>
 <contactref element="U2" pad="16"/>
-<contactref element="U1" pad="1"/>
 <contactref element="LED" pad="K"/>
 <contactref element="C2" pad="2"/>
@@
 <via x="38.354" y="7.62" extent="1-16" drill="0.254"/>
 <via x="33.274" y="2.032" extent="1-16" drill="0.254"/>
+<contactref element="U3" pad="1"/>
 </signal>
 <signal name="VBUS" class="1">
 <contactref element="JP3" pad="3"/>
-<contactref element="U1" pad="3"/>
 <contactref element="USB" pad="1"/>
 <contactref element="C1" pad="1"/>
 <contactref element="R1" pad="2"/>
-<wire x1="13.462" y1="11.43" x2="17.018" y2="14.986" width="0.3048" layer="16"/>
 <wire x1="11.938" y1="14.986" x2="9.144" y2="17.78" width="0.3048" layer="1"/>
 <wire x1="9.144" y1="17.78" x2="8.382" y2="17.78" width="0.3048" layer="1"/>
@@
 <wire x1="15.494" y1="4.826" x2="15.494" y2="6.604" width="0.3048" layer="1"/>
 <via x="15.494" y="6.604" extent="1-16" drill="0.3048"/>
-<wire x1="15.494" y1="6.604" x2="15.494" y2="9.398" width="0.3048" layer="16"/>
-<wire x1="15.494" y1="9.398" x2="13.462" y2="11.43" width="0.3048" layer="16"/>
+<contactref element="U3" pad="2"/>
+<wire x1="14.478" y1="10.668" x2="14.478" y2="7.62" width="0.3048" layer="16"/>
+<wire x1="14.478" y1="7.62" x2="15.494" y2="6.604" width="0.3048" layer="16"/>
+<wire x1="14.478" y1="10.668" x2="14.478" y2="12.446" width="0.3048" layer="16"/>
+<wire x1="14.478" y1="12.446" x2="17.018" y2="14.986" width="0.3048" layer="16"/>
 </signal>
 <signal name="PA04">
@@
 <contactref element="U2" pad="17"/>
 <contactref element="JP1" pad="15"/>
-<contactref element="U1" pad="2"/>
 <contactref element="R3" pad="2"/>
 <contactref element="C2" pad="1"/>
 <contactref element="C3" pad="1"/>
 <contactref element="C4" pad="1"/>
-<wire x1="17.018" y1="12.192" x2="13.716" y2="8.89" width="0.3048" layer="1"/>
-<wire x1="13.462" y1="8.89" x2="13.716" y2="8.89" width="0.3048" layer="1"/>
 <wire x1="17.018" y1="12.192" x2="17.018" y2="9.398" width="0.3048" layer="1"/>
 <wire x1="17.018" y1="12.192" x2="20.8048375" y2="12.192" width="0.3048" layer="16"/>
@@
 <wire x1="35.4584" y1="10.287" x2="33.147" y2="10.287" width="0.3048" layer="1"/>
 <wire x1="33.147" y1="10.287" x2="33.02" y2="10.414" width="0.3048" layer="1"/>
-<wire x1="8.89" y1="1.27" x2="11.3665" y2="3.7465" width="0.3048" layer="1"/>
-<wire x1="11.3665" y1="3.7465" x2="13.34695" y2="3.7465" width="0.3048" layer="1"/>
-<wire x1="13.34695" y1="3.7465" x2="14.7955" y2="5.19505" width="0.3048" layer="1"/>
-<wire x1="14.7955" y1="5.19505" x2="14.7955" y2="7.1755" width="0.3048" layer="1"/>
-<wire x1="14.7955" y1="7.1755" x2="17.018" y2="9.398" width="0.3048" layer="1"/>
+<wire x1="8.89" y1="1.27" x2="17.018" y2="9.398" width="0.3048" layer="1"/>
+<contactref element="U3" pad="3"/>
+<wire x1="11.938" y1="9.398" x2="11.938" y2="9.652" width="0.3048" layer="1"/>
+<wire x1="14.478" y1="12.192" x2="17.018" y2="12.192" width="0.3048" layer="1"/>
+<wire x1="11.938" y1="9.652" x2="14.478" y2="12.192" width="0.3048" layer="1"/>
 </signal>
 <signal name="!RESET">
@@
 <wire x1="47.6238" y1="12.2682" x2="43.0370625" y2="12.2682" width="0.254" layer="1"/>
 <wire x1="43.0370625" y1="12.2682" x2="37.3982625" y2="17.907" width="0.254" layer="1"/>
-<wire x1="11.43" y1="14.224" x2="11.43" y2="6.35" width="0.254" layer="16"/>
-<wire x1="6.35" y1="1.27" x2="11.43" y2="6.35" width="0.254" layer="16"/>
-<wire x1="11.43" y1="14.224" x2="15.113" y2="17.907" width="0.254" layer="16"/>
+<wire x1="10.668" y1="13.462" x2="10.668" y2="5.588" width="0.254" layer="16"/>
+<wire x1="6.35" y1="1.27" x2="10.668" y2="5.588" width="0.254" layer="16"/>
+<wire x1="10.668" y1="13.462" x2="15.113" y2="17.907" width="0.254" layer="16"/>
 <wire x1="30.861" y1="17.907" x2="15.113" y2="17.907" width="0.254" layer="16"/>
 <via x="30.861" y="17.907" extent="1-16" drill="0.254"/>
