File: OSO Curriculum/OSO-SAFE-A1-04.brd (EAGLE design)
At the start: 50.8 x 22.9 mm, 29 parts, among them J1 10118193-0001LF, Q1 DMG341, SW1 SPST_TACT-KMR2, U1 AP2112-3.3, U2 MCP73831T-2ACI/OT, U3 ATSAMD11D14A-SSNT, X1 JSTPH, X2 2x5 0.05" SWD

Commit message: simple samd11 feather a1 rev 04
Parts:
- removed U$7: (no value), My Stuff:OSO_WORDMARK_THREELINE_450MIL_1000DPI
- removed X1: JSTPH, microbuilder:JSTPH2
- added J2: 10118193-0001LF, 10118193-0001LF:FCI_10118193-0001LF
- added TP1, TP2, TP6, TP7, TP8: (no value), microbuilder:TESTPOINT_ROUND_2MM_NO
- added U$9: (no value), My Stuff:OSO_WORDMARK_ONELINE_350MIL_1000DPI
- J1: value 10118193-0001LF -> JSTPH; device 10118193-0001LF:FCI_10118193-0001LF -> microbuilder:JSTPH2
- X2: device microbuilder:2X05_1.27MM_BOX_POSTS -> microbuilder:2X05_1.27MM_BOX_NOPOSTS
- moved J1 12.2 mm to (10.8, 19.3), turned to 0 degrees
Connections:
- net !RESET: now also TP8.P$1
- net +3V3: now also TP1.P$1
- net GND: now also J1.1, J2.5, J2.S1, J2.S2, J2.S3, J2.S4, J2.S5, J2.S6, TP2.P$1; no longer J1.5, J1.S1, J1.S2, J1.S3, J1.S4, J1.S5, J1.S6, X1.1
- net PA30/SWCLK: now also TP6.P$1
- net PA31/SWDIO/LED: now also TP7.P$1
- net USB_N: now also J2.2; no longer J1.2
- net USB_P: now also J2.3; no longer J1.3
- net VBAT: now also J1.2; no longer X1.2
- net VBUS: now also J2.1; no longer J1.1
Routing:
- net +3V3: track 62.3 -> 69.8 mm, vias 3 -> 4
- net PA31/SWDIO/LED: track 56.7 -> 63.7 mm
- net PA30/SWCLK: track 42.3 -> 46.2 mm
- net !RESET: track 59.6 -> 62.2 mm, vias 3 -> 4
Other:
- board text added: "!RESET"
- board text added: "10µF 1µF 100KΩ 10KΩ 1KΩ"
- board text added: "A0 PA02"
- board text added: "A1 PA04"
- board text added: "A2 PA05"
- board text added: "A3 PA06"
- board text added: "A4 PA07"
- board text added: "PA08 11"
- board text added: "PA09 10"
- board text added: "PA14 SDA"
- board text added: "PA15 SCL"
- board text added: "PA16 9"
- board text added: "PA22 6"
- board text added: "PA23 5"
- board text added: "PA30 12/SWCLK"
- board text added: "PA31/LED 13/SWDIO"
- board text added: "PARTS LIST"
- board text added: "Pins 5, 6, 9, 10, & 11 are duplicated on the top and bottom rows to support more wings. Use as SPI/UART or GPIO, but not both."
- board text added: "SW1"
- board text added: "SWCLK"
- board text added: "SWDIO"
- board text added: "Simple Surface-Mount SAM D11 Feather OSO-SAFE-A1-04"
- board text added: "U1: AP2112K-3.3 U2: MCP73831T-2ACI/OT U3: ATSAMD11D14AS C1 C2 C4 C5........ C3 C6.................... R1.......................... R2 R4 R5.............. R3 R6.................... D1: MBR120; Q1: DMG3415 LED/CHG: 0805 LEDs with VF=2V, like LTST-C171KRKT/KSKT SW1: KMR231NG J1: S2B-PH-SM4 J2: 10118193"
- board text added: "U3 is a SAM D11 20-pin SOIC. The brains of the operation! C5 filters power, C6 smooths out AREF. R5 is a pull-up for SWCLK. Aside from USB, all the other pins fan out to the Feather headers."
- board text removed: "@josecastillo"
- board text removed: "AIN PA04"
- board text removed: "AIN PA05"
- board text removed: "AIN PA06"
- board text removed: "AIN PA07"
- board text removed: "AIN/VOUT PA02"
- board text removed: "NC"
- board text removed: "PA08"
- board text removed: "PA08, 09, 16, 22 and 23 are duplicated on the top row to support more wings; use as SPI/UART or GPIO, but not both."
- board text removed: "PA09"
- board text removed: "PA16"
- board text removed: "PA22"
- board text removed: "PA23"
- board text removed: "PA30 SWCLK"
- board text removed: "PA31/LED SWDIO"
- board text removed: "Road to the Book #6 oddlyspecific.org"
- board text removed: "SCL PA15"
- board text removed: "SDA PA14"
- board text removed: "Simple Surface-Mount SAM D11 Feather OSO-SAFE-A1-03"
- board text removed: "U3 is a SAM D11 20-pin SOIC. The brains of the operation! C5 filters power, C6 smooths out AREF. R5 is a pull-up for SWCLK. Aside from USB, the rest of the pins fan out to the Feather headers."
