File: OSO Curriculum/OSO-SAFE-A1-04.sch (EAGLE design)
At the start: 27 parts, among them J1 10118193-0001LF, Q1 DMG341, SW1 SPST_TACT-KMR2, U1 AP2112-3.3, U2 MCP73831T-2ACI/OT, U3 ATSAMD11D14A-SSNT, X1 JSTPH, X2 2x5 0.05" SWD

Commit message: simple samd11 feather a1 rev 04
Parts:
- removed X1: JSTPH, microbuilder:CON_JST_PH_2PIN
- added J2: 10118193-0001LF, 10118193-0001LF:10118193-0001LF
- added TP1, TP2, TP6, TP7, TP8: (no value), microbuilder:TESTPOINTROUND2MMNO
- J1: value 10118193-0001LF -> JSTPH; device 10118193-0001LF:10118193-0001LF -> microbuilder:CON_JST_PH_2PIN
- X2: device microbuilder:JTAG-CORTEXBOXPOSTS -> microbuilder:JTAG-CORTEXBOX
Connections:
- net !RESET: now also TP8.P$1
- net +3V3: now also TP1.P$1
- net GND: now also J1.1, J2.GND, J2.SHIELD, TP2.P$1; no longer J1.GND, J1.SHIELD, X1.1
- net PA30/SWCLK: now also TP6.P$1
- net PA31/SWDIO/LED: now also TP7.P$1
- net USB_N: now also J2.D-; no longer J1.D-
- net USB_P: now also J2.D+; no longer J1.D+
- net VBAT: now also J1.2; no longer X1.2
- net VBUS: now also J2.VUSB; no longer J1.VUSB
Other:
- moved on the sheet: C4, C6, CHG, JP2, JP4, LED, R3, R4, R5, R6, U2, U3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
