File: Temperature Hat/Daughterboards/OSO-MISC-20-004 Pulse Oximetry.brd (EAGLE design)
At the start: 19.8 x 12.7 mm, 13 parts, among them J1 SM03B-SRSS-TB(LF)(SN), U1 LIGHT_SENSOR1206

Commit message: add led resistor values
Parts:
- R2: value TBD -> 220
- R4: value TBD -> 120
Changed lines of the file:
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@@
 <layers>
 <layer number="1" name="Top" color="4" fill="1" visible="yes" active="yes"/>
-<layer number="2" name="Route2" color="16" fill="1" visible="yes" active="yes"/>
-<layer number="3" name="Route3" color="17" fill="1" visible="yes" active="yes"/>
-<layer number="4" name="Route4" color="18" fill="1" visible="yes" active="yes"/>
-<layer number="5" name="Route5" color="19" fill="1" visible="yes" active="yes"/>
-<layer number="6" name="Route6" color="25" fill="1" visible="yes" active="yes"/>
-<layer number="7" name="Route7" color="26" fill="1" visible="yes" active="yes"/>
-<layer number="8" name="Route8" color="27" fill="1" visible="yes" active="yes"/>
-<layer number="9" name="Route9" color="28" fill="1" visible="yes" active="yes"/>
-<layer number="10" name="Route10" color="29" fill="1" visible="yes" active="yes"/>
-<layer number="11" name="Route11" color="30" fill="1" visible="yes" active="yes"/>
-<layer number="12" name="Route12" color="20" fill="1" visible="yes" active="yes"/>
-<layer number="13" name="Route13" color="21" fill="1" visible="yes" active="yes"/>
-<layer number="14" name="Route14" color="22" fill="1" visible="yes" active="yes"/>
-<layer number="15" name="Route15" color="23" fill="1" visible="yes" active="yes"/>
-<layer number="16" name="Bottom" color="1" fill="1" visible="yes" active="yes"/>
+<layer number="2" name="Route2" color="16" fill="1" visible="no" active="yes"/>
+<layer number="3" name="Route3" color="17" fill="1" visible="no" active="yes"/>
+<layer number="4" name="Route4" color="18" fill="1" visible="no" active="yes"/>
+<layer number="5" name="Route5" color="19" fill="1" visible="no" active="yes"/>
+<layer number="6" name="Route6" color="25" fill="1" visible="no" active="yes"/>
+<layer number="7" name="Route7" color="26" fill="1" visible="no" active="yes"/>
+<layer number="8" name="Route8" color="27" fill="1" visible="no" active="yes"/>
+<layer number="9" name="Route9" color="28" fill="1" visible="no" active="yes"/>
+<layer number="10" name="Route10" color="29" fill="1" visible="no" active="yes"/>
+<layer number="11" name="Route11" color="30" fill="1" visible="no" active="yes"/>
+<layer number="12" name="Route12" color="20" fill="1" visible="no" active="yes"/>
+<layer number="13" name="Route13" color="21" fill="1" visible="no" active="yes"/>
+<layer number="14" name="Route14" color="22" fill="1" visible="no" active="yes"/>
+<layer number="15" name="Route15" color="23" fill="1" visible="no" active="yes"/>
+<layer number="16" name="Bottom" color="1" fill="1" visible="no" active="yes"/>
 <layer number="17" name="Pads" color="2" fill="1" visible="yes" active="yes"/>
 <layer number="18" name="Vias" color="2" fill="1" visible="yes" active="yes"/>
@@
 <layer number="20" name="Dimension" color="24" fill="1" visible="yes" active="yes"/>
 <layer number="21" name="tPlace" color="7" fill="1" visible="yes" active="yes"/>
-<layer number="22" name="bPlace" color="7" fill="1" visible="yes" active="yes"/>
+<layer number="22" name="bPlace" color="7" fill="1" visible="no" active="yes"/>
 <layer number="23" name="tOrigins" color="15" fill="1" visible="yes" active="yes"/>
-<layer number="24" name="bOrigins" color="15" fill="1" visible="yes" active="yes"/>
+<layer number="24" name="bOrigins" color="15" fill="1" visible="no" active="yes"/>
 <layer number="25" name="tNames" color="7" fill="1" visible="yes" active="yes"/>
-<layer number="26" name="bNames" color="7" fill="1" visible="yes" active="yes"/>
+<layer number="26" name="bNames" color="7" fill="1" visible="no" active="yes"/>
 <layer number="27" name="tValues" color="7" fill="1" visible="no" active="yes"/>
 <layer number="28" name="bValues" color="7" fill="1" visible="no" active="yes"/>
@@
 <layer number="38" name="bTest" color="7" fill="1" visible="no" active="yes"/>
 <layer number="39" name="tKeepout" color="4" fill="11" visible="yes" active="yes"/>
-<layer number="40" name="bKeepout" color="1" fill="11" visible="yes" active="yes"/>
+<layer number="40" name="bKeepout" color="1" fill="11" visible="no" active="yes"/>
 <layer number="41" name="tRestrict" color="4" fill="10" visible="yes" active="yes"/>
-<layer number="42" name="bRestrict" color="1" fill="10" visible="yes" active="yes"/>
+<layer number="42" name="bRestrict" color="1" fill="10" visible="no" active="yes"/>
 <layer number="43" name="vRestrict" color="2" fill="10" visible="no" active="yes"/>
 <layer number="44" name="Drills" color="7" fill="1" visible="no" active="yes"/>
@@
 <layer number="50" name="dxf" color="7" fill="1" visible="no" active="no"/>
 <layer number="51" name="tDocu" color="7" fill="1" visible="yes" active="yes"/>
-<layer number="52" name="bDocu" color="7" fill="1" visible="yes" active="yes"/>
+<layer number="52" name="bDocu" color="7" fill="1" visible="no" active="yes"/>
 <layer number="53" name="tGND_GNDA" color="7" fill="9" visible="no" active="no"/>
 <layer number="54" name="bGND_GNDA" color="1" fill="9" visible="no" active="no"/>
@@
 <attribute name="VALUE" x="5.30225" y="6.35" size="0.508" layer="28" font="vector" ratio="18" rot="MR90" align="center"/>
 </element>
-<element name="R2" library="microbuilder" package="0805-NO" value="TBD" x="8.636" y="7.366" smashed="yes" rot="R180">
+<element name="R2" library="microbuilder" package="0805-NO" value="220" x="8.636" y="7.366" smashed="yes" rot="R180">
 <attribute name="NAME" x="10.668" y="7.366" size="0.508" layer="25" font="vector" ratio="18" rot="R270" align="center"/>
 <attribute name="VALUE" x="6.604" y="8.128" size="0.508" layer="27" font="vector" ratio="18" rot="R180" align="center"/>
 </element>
-<element name="R4" library="microbuilder" package="0805-NO" value="TBD" x="8.636" y="5.334" smashed="yes" rot="R180">
+<element name="R4" library="microbuilder" package="0805-NO" value="120" x="8.636" y="5.334" smashed="yes" rot="R180">
 <attribute name="NAME" x="10.668" y="5.334" size="0.508" layer="25" font="vector" ratio="18" rot="R270" align="center"/>
 <attribute name="VALUE" x="6.604" y="6.096" size="0.508" layer="27" font="vector" ratio="18" rot="R180" align="center"/>

Commit message: add part numbers
Parts:
- D1: value XZM2CRKM2DGFBB45SCCB -> XZM2MRTNI45SC2C
- U1: value LIGHT_SENSOR1206 -> PT15-21C
Changed lines of the file:
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@@
 <attribute name="VALUE" x="6.604" y="10.668" size="0.508" layer="27" font="vector" ratio="18" rot="R180" align="center"/>
 </element>
-<element name="D1" library="My Stuff" package="PLCC4SMDLED" value="XZM2CRKM2DGFBB45SCCB" x="3.556" y="6.35" smashed="yes" rot="MR270">
+<element name="D1" library="My Stuff" package="PLCC4SMDLED" value="XZM2MRTNI45SC2C" x="3.556" y="6.35" smashed="yes" rot="MR270">
 <attribute name="NAME" x="1.80975" y="6.35" size="0.508" layer="26" font="vector" ratio="18" rot="MR270" align="center"/>
 <attribute name="PROD_ID" value="DIO-13722" x="3.556" y="6.35" size="1.778" layer="28" rot="MR270" display="off"/>
@@
 <attribute name="VALUE" x="6.604" y="6.096" size="0.508" layer="27" font="vector" ratio="18" rot="R180" align="center"/>
 </element>
-<element name="U1" library="SparkFun-Sensors" package="LED-1206" value="LIGHT_SENSOR1206" x="6.35" y="6.604" smashed="yes" rot="MR90">
+<element name="U1" library="SparkFun-Sensors" package="LED-1206" value="PT15-21C" x="6.35" y="6.604" smashed="yes" rot="MR90">
 <attribute name="NAME" x="7.5565" y="6.604" size="0.508" layer="26" font="vector" ratio="18" rot="MR90" align="center"/>
 <attribute name="VALUE" x="5.3975" y="6.604" size="0.508" layer="28" font="vector" ratio="18" rot="MR90" align="center"/>
