File: Totally Not Feather Related/OSO-MISC-20-018 Memory Gadget.brd (EAGLE design)
At the start: 48.3 x 92.7 mm, 58 parts, among them IC1 LS013B4DN04, IC2 S-882150APH, IC3 ATSAMD21G18_QFN, J2 10118193-0001LF, J4 SM04B-SRSS-TB(LF)(SN), Q1 DMG341, SW1 JS102011SAQN, SW2 SPST_TACT-KMR2, U1 MCP73831T-2ACI/OT, U2 AP2112K-3.3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

Commit message: add EN pull-up, fix SPI flash pin selection
Parts:
- added R9: 100K, microbuilder:0805-NO
Connections:
- net EN: now also R9.1
- net FLASHMISO: now also IC3.27; no longer IC3.23
- net V+: now also R9.2
Routing:
- net FLASHMISO: track 17.1 -> 25.8 mm, vias 2 -> 4
Changed lines of the file:
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@@
 </element>
 <element name="U$16" library="My Stuff" package="OSO_WORDMARK_THREELINE_450MIL_1000DPI" value="" x="34.798" y="-16.256" smashed="yes"/>
+<element name="R9" library="microbuilder" package="0805-NO" value="100K" x="-8.89" y="-93.98" smashed="yes">
+<attribute name="NAME" x="-6.858" y="-94.107" size="0.8128" layer="25" ratio="18"/>
+<attribute name="VALUE" x="-6.858" y="-94.742" size="0.4064" layer="27" ratio="10"/>
+</element>
 </elements>
 <signals>
@@
 <wire x1="19.078" y1="-61.5" x2="19.28285" y2="-61.70485" width="0.254" layer="1"/>
 <via x="19.28285" y="-61.70485" extent="1-16" drill="0.254"/>
-<wire x1="40.62285" y1="-53.83085" x2="27.15685" y2="-53.83085" width="0.254" layer="16"/>
-<wire x1="19.28285" y1="-61.70485" x2="27.15685" y2="-53.83085" width="0.254" layer="16"/>
-<wire x1="40.62285" y1="-53.83085" x2="41.402" y2="-54.61" width="0.254" layer="16"/>
+<wire x1="40.64825" y1="-53.85625" x2="27.13145" y2="-53.85625" width="0.254" layer="16"/>
+<wire x1="19.28285" y1="-61.70485" x2="27.13145" y2="-53.85625" width="0.254" layer="16"/>
+<wire x1="40.64825" y1="-53.85625" x2="41.402" y2="-54.61" width="0.254" layer="16"/>
 <via x="41.402" y="-54.61" extent="1-16" drill="0.254"/>
 <wire x1="41.402" y1="-54.61" x2="41.592" y2="-54.42" width="0.254" layer="1"/>
@@
 <via x="12.921" y="-48.735" extent="1-16" drill="0.3048"/>
 <wire x1="7.112" y1="-36.576" x2="7.112" y2="-42.926" width="0.3048" layer="16"/>
+<contactref element="R9" pad="2"/>
+<wire x1="11.872" y1="-49.784" x2="-7.94" y2="-93.98" width="0" layer="19" extent="1-1"/>
 </signal>
 <signal name="VBUS" class="1">
@@
 <wire x1="4.528" y1="-12.192" x2="7.8781" y2="-12.192" width="0.3048" layer="1"/>
 <wire x1="7.8781" y1="-12.192" x2="14.1001" y2="-18.414" width="0.3048" layer="1"/>
+<contactref element="R9" pad="1"/>
+<wire x1="14.1001" y1="-18.414" x2="-9.84" y2="-93.98" width="0" layer="19" extent="1-1"/>
 </signal>
 <signal name="N$2">
@@
 </signal>
 <signal name="FLASHMISO">
-<contactref element="IC3" pad="23"/>
 <contactref element="U3" pad="2"/>
-<wire x1="24.303" y1="-54.646" x2="28.4146" y2="-54.646" width="0.254" layer="1"/>
-<wire x1="28.4146" y1="-54.646" x2="28.448" y2="-54.6126" width="0.254" layer="1"/>
 <via x="28.448" y="-54.6126" extent="1-16" drill="0.254"/>
 <wire x1="28.448" y1="-54.6126" x2="28.956" y2="-55.1206" width="0.254" layer="16"/>
@@
 <wire x1="30.099" y1="-64.643" x2="32.318" y2="-64.643" width="0.254" layer="1"/>
 <wire x1="28.956" y1="-55.1206" x2="28.956" y2="-63.5" width="0.254" layer="16"/>
+<contactref element="IC3" pad="27"/>
+<via x="24.5618" y="-49.53" extent="1-16" drill="0.254"/>
+<wire x1="22.578" y1="-53.421" x2="22.578" y2="-52.59834375" width="0.254" layer="1"/>
+<wire x1="22.578" y1="-52.59834375" x2="22.6314" y2="-52.54494375" width="0.254" layer="1"/>
+<wire x1="23.68045625" y1="-49.125" x2="24.17314375" y2="-49.125" width="0.254" layer="1"/>
+<wire x1="24.5618" y1="-49.53" x2="24.5618" y2="-49.51365625" width="0.254" layer="1"/>
+<wire x1="24.5618" y1="-49.51365625" x2="24.17314375" y2="-49.125" width="0.254" layer="1"/>
+<wire x1="22.6314" y1="-52.54494375" x2="22.6314" y2="-51.64648125" width="0.254" layer="1"/>
+<wire x1="22.6314" y1="-51.64648125" x2="22.4282" y2="-51.44328125" width="0.254" layer="1"/>
+<wire x1="22.4282" y1="-51.44328125" x2="22.4282" y2="-50.37725625" width="0.254" layer="1"/>
+<wire x1="22.4282" y1="-50.37725625" x2="23.68045625" y2="-49.125" width="0.254" layer="1"/>
+<wire x1="24.5618" y1="-49.53" x2="24.80755" y2="-49.53" width="0.254" layer="16"/>
+<wire x1="28.194" y1="-52.91645" x2="24.80755" y2="-49.53" width="0.254" layer="16"/>
+<wire x1="28.194" y1="-52.91645" x2="28.2194" y2="-52.91645" width="0.254" layer="16"/>
+<via x="28.2194" y="-52.91645" extent="1-16" drill="0.254"/>
+<wire x1="28.2194" y1="-52.91645" x2="28.321" y2="-53.01805" width="0.254" layer="1"/>
+<wire x1="28.321" y1="-53.01805" x2="28.321" y2="-54.4856" width="0.254" layer="1"/>
+<wire x1="28.321" y1="-54.4856" x2="28.448" y2="-54.6126" width="0.254" layer="1"/>
 </signal>
 <signal name="FLASHCS">
