File: SAML22 Feather/OSO-MISC-21-005 SAML22 Feather.brd (EAGLE design)
At the start: 50.8 x 22.9 mm, 46 parts, among them J1 JSTPH, J2 10118193-0001LF, J3 2x5 0.05" SWD, Q1 DMG341, SW1 SPST_TACT-KMR2, U1 AP2112-3.3, U2 MCP73831T-2ACI/OT, U3 ATSAML22J18A-MUT, X1 32khz/7pF

Commit message: saml22 feather: rename segment pins for clarity
Connections:
- net SEG2: now also U$6.P$4, U3.19; no longer U$6.P$6, U3.24
- net SEG3: now also U$6.P$5, U3.20; no longer U$6.P$17, U3.25
- net SEG4: now also U$6.P$6, U3.24; no longer U$6.P$18, U3.26
- net SEG5: now also U$6.P$17, U3.25; no longer U$6.P$7, U3.27
- net SEG6: now also U$6.P$18, U3.26; no longer U$6.P$8, U3.28
- net SEG7: now also U$6.P$7, U3.27; no longer U$6.P$4, U3.19
- net SEG8: now also U$6.P$8, U3.28; no longer U$6.P$5, U3.20
Routing:
- net SEG5: track 9.19 -> 19.2 mm
- net SEG6: track 8.89 -> 18.6 mm
- net SEG4: track 18.6 -> 10.7 mm
- net SEG3: track 19.2 -> 12.7 mm
- net SEG7: track 13.6 -> 9.19 mm
- net SEG8: track 12.7 -> 8.89 mm
- net SEG2: track 10.7 -> 13.6 mm
Changed lines of the file:
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@@
 <drawing>
 <settings>
-<setting alwaysvectorfont="yes"/>
+<setting alwaysvectorfont="no"/>
 <setting keepoldvectorfont="yes"/>
 <setting verticaltext="up"/>
@@
 <wire x1="33.810475" y1="13.1333875" x2="36.918" y2="16.2409125" width="0.1524" layer="1"/>
 </signal>
-<signal name="SEG8">
+<signal name="SEG3">
 <contactref element="U3" pad="20"/>
 <contactref element="U$6" pad="P$5"/>
@@
 <wire x1="22.5242" y1="13.2209375" x2="22.5242" y2="14.6258" width="0.1524" layer="1"/>
 </signal>
-<signal name="SEG7">
+<signal name="SEG2">
 <contactref element="U3" pad="19"/>
 <contactref element="U$6" pad="P$4"/>
@@
 <wire x1="23.6728" y1="9.483025" x2="23.6728" y2="5.75931875" width="0.1524" layer="1"/>
 </signal>
-<signal name="SEG2">
+<signal name="SEG4">
 <contactref element="U3" pad="24"/>
 <wire x1="23.248225" y1="13.2153375" x2="23.248225" y2="12.4787375" width="0.1524" layer="16"/>
@@
 <wire x1="24.8263625" y1="9.402" x2="23.857825" y2="10.3705375" width="0.1524" layer="16"/>
 </signal>
-<signal name="SEG3">
+<signal name="SEG5">
 <contactref element="U3" pad="25"/>
 <wire x1="25.8318" y1="9.902" x2="24.7581625" y2="9.902" width="0.1524" layer="16"/>
@@
 <wire x1="33.93673125" y1="12.8285875" x2="38.118" y2="17.00985625" width="0.1524" layer="1"/>
 </signal>
-<signal name="SEG4">
+<signal name="SEG6">
 <contactref element="U3" pad="26"/>
 <wire x1="24.9947625" y1="10.402" x2="24.975425" y2="10.4213375" width="0.1524" layer="16"/>
@@
 <wire x1="34.0433375" y1="12.5041375" x2="37.3986" y2="15.8594" width="0.1524" layer="1"/>
 </signal>
-<signal name="SEG5">
+<signal name="SEG7">
 <contactref element="U3" pad="27"/>
 <via x="23.756225" y="12.7073375" extent="1-16" drill="0.3048"/>
@@
 <wire x1="26.162" y1="16.0274" x2="23.7942" y2="13.6596" width="0.1524" layer="1"/>
 </signal>
-<signal name="SEG6">
+<signal name="SEG8">
 <contactref element="U3" pad="28"/>
 <via x="24.467425" y="12.6311375" extent="1-16" drill="0.3048"/>
