File: SAML22 Feather/OSO-MISC-21-005 SAML22 Feather.sch (EAGLE design)
At the start: 44 parts, among them J1 JSTPH, J2 10118193-0001LF, J3 2x5 0.05" SWD, Q1 DMG341, SW1 SPST_TACT-KMR2, U1 AP2112-3.3, U2 MCP73831T-2ACI/OT, U3 ATSAML22J18A-MUT, X1 32khz/7pF

Commit message: saml22 feather: rename segment pins for clarity
Connections:
- net SEG2: now also U$6.P$4, U3A.PA10/I10/SERCOM0.2/SLCD[13]; no longer U$6.P$6, U3A.PB11/I11/SERCOM3.3/SLCD[21]
- net SEG3: now also U$6.P$5, U3A.PA11/I11/SERCOM0.3/SLCD[14]; no longer U$6.P$17, U3A.PB12/I12/SERCOM3.0/SLCD[22]
- net SEG4: now also U$6.P$6, U3A.PB11/I11/SERCOM3.3/SLCD[21]; no longer U$6.P$18, U3A.PB13/SERCOM3.1/SLCD[23]
- net SEG5: now also U$6.P$17, U3A.PB12/I12/SERCOM3.0/SLCD[22]; no longer U$6.P$7, U3A.PB14/I14/SERCOM3.2/SLCD[24]
- net SEG6: now also U$6.P$18, U3A.PB13/SERCOM3.1/SLCD[23]; no longer U$6.P$8, U3A.PB15/I15/SERCOM3.3/SLCD[25]
- net SEG7: now also U$6.P$7, U3A.PB14/I14/SERCOM3.2/SLCD[24]; no longer U$6.P$4, U3A.PA10/I10/SERCOM0.2/SLCD[13]
- net SEG8: now also U$6.P$8, U3A.PB15/I15/SERCOM3.3/SLCD[25]; no longer U$6.P$5, U3A.PA11/I11/SERCOM0.3/SLCD[14]
Other:
- note added: "LIQUID CRYSTAL DISPLAY"
- note added: "SAM L22 MICROCONTROLLER"
- note added: "SAM L22 POWER"
- note added: "SWD CONNECTOR"
- note added: "USB PORT"
- moved on the sheet: C10, C11, C12, C13, C14, C4, C5, C6, C7, C8, C9, CHG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
